Commit message: add description

File: manipulator_description/urdf/manipulator.xacro (robot description, xacro)
@@ -4,4 +4,6 @@
 <xacro:include filename="$(find manipulator_description)/urdf/manipulator.trans" />
 <xacro:include filename="$(find manipulator_description)/urdf/manipulator.gazebo" />
+<link name="dummy">
+</link>
 <link name="base_link">
   <inertial>
@@ -15,5 +17,5 @@
       <mesh filename="package://manipulator_description/meshes/base_link.stl" scale="0.001 0.001 0.001"/>
     </geometry>
-    <material name="silver_default"/>
+    <material name="yellow"/>
   </visual>
   <collision>
@@ -35,5 +37,5 @@
       <mesh filename="package://manipulator_description/meshes/S3003_v5_1.stl" scale="0.001 0.001 0.001"/>
     </geometry>
-    <material name="silver_default"/>
+    <material name="black"/>
   </visual>
   <collision>
@@ -55,5 +57,5 @@
       <mesh filename="package://manipulator_description/meshes/bottom_linkz_v4_1.stl" scale="0.001 0.001 0.001"/>
     </geometry>
-    <material name="silver_default"/>
+    <material name="yellow"/>
   </visual>
   <collision>
@@ -75,5 +77,5 @@
       <mesh filename="package://manipulator_description/meshes/S3003_v5_2.stl" scale="0.001 0.001 0.001"/>
     </geometry>
-    <material name="silver_default"/>
+    <material name="black"/>
   </visual>
   <collision>
@@ -95,5 +97,5 @@
       <mesh filename="package://manipulator_description/meshes/link_v3_1.stl" scale="0.001 0.001 0.001"/>
     </geometry>
-    <material name="silver_default"/>
+    <material name="yellow"/>
   </visual>
   <collision>
@@ -115,5 +117,5 @@
       <mesh filename="package://manipulator_description/meshes/S3003_v5_3.stl" scale="0.001 0.001 0.001"/>
     </geometry>
-    <material name="silver_default"/>
+    <material name="black"/>
   </visual>
   <collision>
@@ -135,5 +137,5 @@
       <mesh filename="package://manipulator_description/meshes/link_v3_2.stl" scale="0.001 0.001 0.001"/>
     </geometry>
-    <material name="silver_default"/>
+    <material name="yellow"/>
   </visual>
   <collision>
@@ -155,5 +157,5 @@
       <mesh filename="package://manipulator_description/meshes/S3003_v5_4.stl" scale="0.001 0.001 0.001"/>
     </geometry>
-    <material name="silver_default"/>
+    <material name="black"/>
   </visual>
   <collision>
@@ -175,5 +177,5 @@
       <mesh filename="package://manipulator_description/meshes/hand_front_v1_1.stl" scale="0.001 0.001 0.001"/>
     </geometry>
-    <material name="silver_default"/>
+    <material name="yellow"/>
   </visual>
   <collision>
@@ -195,5 +197,5 @@
       <mesh filename="package://manipulator_description/meshes/hand_back_v1_1.stl" scale="0.001 0.001 0.001"/>
     </geometry>
-    <material name="silver_default"/>
+    <material name="yellow"/>
   </visual>
   <collision>
@@ -295,5 +297,5 @@
       <mesh filename="package://manipulator_description/meshes/finger_v1_1.stl" scale="0.001 0.001 0.001"/>
     </geometry>
-    <material name="silver_default"/>
+    <material name="red"/>
   </visual>
   <collision>
@@ -315,5 +317,5 @@
       <mesh filename="package://manipulator_description/meshes/finger_v1_2.stl" scale="0.001 0.001 0.001"/>
     </geometry>
-    <material name="silver_default"/>
+    <material name="red"/>
   </visual>
   <collision>
@@ -324,4 +326,8 @@
   </collision>
 </link>
+<joint name="dummy_joint" type="fixed">
+ <parent link="dummy"/>
+ <child link="base_link"/>
+</joint>
 <joint name="Rigid1" type="fixed">
   <origin rpy="0 0 0" xyz="-0.005025 0.009822 0.003022"/>
@@ -329,9 +335,10 @@
   <child link="S3003_v5_1"/>
 </joint>
-<joint name="Rev2" type="continuous">
+<joint name="Rev2" type="revolute">
   <origin rpy="0 0 0" xyz="0.005025 -0.013844 0.01641"/>
   <parent link="S3003_v5_1"/>
   <child link="bottom_linkz_v4_1"/>
   <axis xyz="-0.0 0.015707 0.999877"/>
+  <limit effort="30" lower="-2.617" upper="2.617" velocity="1.571"/>
 </joint>
 <joint name="Rigid3" type="fixed">
@@ -340,9 +347,10 @@
   <child link="S3003_v5_2"/>
 </joint>
-<joint name="Rev4" type="continuous">
+<joint name="Rev4" type="revolute">
   <origin rpy="0 0 0" xyz="-0.0141 0.016267 0.00477"/>
   <parent link="S3003_v5_2"/>
   <child link="link_v3_1"/>
   <axis xyz="-0.0 0.999877 -0.015707"/>
+  <limit effort="30" lower="-2.617" upper="2.617" velocity="1.571"/>
 </joint>
 <joint name="Rigid5" type="fixed">
@@ -351,9 +359,10 @@
   <child link="S3003_v5_3"/>
 </joint>
-<joint name="Rev6" type="continuous">
+<joint name="Rev6" type="revolute">
   <origin rpy="0 0 0" xyz="-0.005025 0.015967 -0.014353"/>
   <parent link="S3003_v5_3"/>
   <child link="link_v3_2"/>
   <axis xyz="-0.0 0.999877 -0.015707"/>
+  <limit effort="30" lower="-2.617" upper="2.617" velocity="1.571"/>
 </joint>
 <joint name="Rigid7" type="fixed">
@@ -362,9 +371,10 @@
   <child link="S3003_v5_4"/>
 </joint>
-<joint name="Rev8" type="continuous">
+<joint name="Rev8" type="revolute">
   <origin rpy="0 0 0" xyz="0.005025 0.015966 -0.014353"/>
   <parent link="S3003_v5_4"/>
   <child link="hand_front_v1_1"/>
   <axis xyz="-0.0 0.999877 -0.015707"/>
+  <limit effort="30" lower="-2.617" upper="2.617" velocity="1.571"/>
 </joint>
 <joint name="Rigid9" type="fixed">
@@ -373,39 +383,45 @@
   <child link="hand_back_v1_1"/>
 </joint>
-<joint name="Rev10" type="continuous">
+<joint name="Rev10" type="revolute">
   <origin rpy="0 0 0" xyz="0.01 -0.013728 0.004717"/>
   <parent link="hand_back_v1_1"/>
   <child link="hand_right_branch_v2_1"/>
   <axis xyz="-1.0 -0.0 -0.0"/>
-</joint>
-<joint name="Rev11" type="continuous">
+  <limit effort="30" lower="-2.617" upper="0" velocity="1.571"/>
+</joint>
+<joint name="Rev11" type="revolute">
   <origin rpy="0 0 0" xyz="0.01 0.013869 0.004283"/>
   <parent link="hand_back_v1_1"/>
   <child link="hand_left_branch_v1_1"/>
   <axis xyz="-1.0 -0.0 -0.0"/>
-</joint>
-<joint name="Rev12" type="continuous">
+  <limit effort="30" lower="0" upper="2.617" velocity="1.571"/>
+</joint>
+<joint name="Rev12" type="revolute">
   <origin rpy="0 0 0" xyz="0.01 -0.00843 0.023097"/>
   <parent link="hand_back_v1_1"/>
   <child link="hand_right_branch_child_v1_1"/>
   <axis xyz="-1.0 -0.0 -0.0"/>
-</joint>
-<joint name="Rev13" type="continuous">
+  <limit effort="30" lower="-2.617" upper="2.617" velocity="1.571"/>
+</joint>
+<joint name="Rev13" type="revolute">
   <origin rpy="0 0 0" xyz="0.01 0.009152 0.02282"/>
   <parent link="hand_back_v1_1"/>
   <child link="hand_left_branch_child_v1_1"/>
   <axis xyz="-1.0 -0.0 -0.0"/>
-</joint>
-<joint name="Rev14" type="continuous">
+  <limit effort="30" lower="-2.617" upper="2.617" velocity="1.571"/>
+</joint>
+<joint name="Rev14" type="revolute">
   <origin rpy="0 0 0" xyz="-0.0058 0.000519 0.032995"/>
   <parent link="hand_right_branch_v2_1"/>
   <child link="finger_v1_1"/>
   <axis xyz="-1.0 -0.0 -0.0"/>
-</joint>
-<joint name="Rev16" type="continuous">
+  <limit effort="30" lower="-2.617" upper="2.617" velocity="1.571"/>
+</joint>
+<joint name="Rev15" type="revolute">
   <origin rpy="0 0 0" xyz="-0.0058 0.00023 0.032999"/>
   <parent link="hand_left_branch_v1_1"/>
   <child link="finger_v1_2"/>
   <axis xyz="-1.0 0.0 -0.0"/>
+  <limit effort="30" lower="-2.617" upper="2.617" velocity="1.571"/>
 </joint>
 </robot>

File: manipulator_description/urdf/materials.xacro (robot description, xacro)
@@ -1,4 +1,22 @@
 <?xml version="1.0" ?>
 <robot name="manipulator" xmlns:xacro="http://www.ros.org/wiki/xacro" >
+<material name="red">
+    <color rgba="1.0 0.0 0.0 1.0"/>
+</material>
+<material name="green">
+    <color rgba="0.0 1.0 0.0 1.0"/>
+</material>
+<material name="blue">
+    <color rgba="0.0 0.0 1.0 1.0"/>
+</material>
+<material name="yellow">
+    <color rgba="1.0 1.0 0.0 1.0"/>
+</material>
+<material name="black">
+    <color rgba="0.0 0.0 0.0 1.0"/>
+</material>
+<material name="white">
+    <color rgba="1.0 1.0 1.0 1.0"/>
+</material>
 <material name="silver_default">
   <color rgba="0.700 0.700 0.700 1.000"/>
